File: hardware/PCB/TFG_PCB/TFG_PCB.sch (KiCad schematic (older format))
At the start: 48 parts, among them J1 Conn_01x02_Male, J10 Conn_01x02_Male, J2 Conn_01x04_Male, J3 Conn_01x04_Male, J4 Conn_01x02_Male, J5 Conn_01x02_Male, J6 Conn_01x02_Male, J7 Conn_01x04_Male, J8 Conn_01x04_Male, J9 Conn_01x02_Male, Q1 FDD6685, Q2 FDD6685, Q3 2N7002, U1 L78L05_SOT89, U2 TD7590_2, U3 TD7590_2

Commit message: Added hierarchy and logic sheet
Parts:
- removed C1, C10, C2, C9: 10u, symbol Device:C
- removed C3, C4, C5, C6, C7, C8: 470u, symbol Device:C
- removed D1, D2: SDT5100LP5-13, SDT5100LP513, symbol SamacSys_Parts:SDT5100LP5-13
- removed J1, J10, J4, J5, J6, J9, J? (x3): Conn_01x02_Male, symbol Connector:Conn_01x02_Male
- removed J2, J3, J7, J8, J? (x2): Conn_01x04_Male, symbol Connector:Conn_01x04_Male
- removed L1, L2: 15u, symbol Device:L
- removed Q1, Q2: FDD6685, FQD1N80TM, symbol SamacSys_Parts:FDD6685
- removed Q3: 2N7002, Package_TO_SOT_SMD:SOT-23, symbol Transistor_FET:2N7002
- removed Q?: IRF540N, Package_TO_SOT_THT:TO-220-3_Vertical, symbol Transistor_FET:IRF540N
- removed R1, R10, R11, R2, R3, R?: 10k, symbol Device:R
- removed R4, R5: 100k, symbol Device:R
- removed R6: 300k, symbol Device:R
- removed R7: 68k, symbol Device:R
- removed R8: 47k, symbol Device:R
- removed R9: 22k, symbol Device:R
- removed U1: L78L05_SOT89, Package_TO_SOT_SMD:SOT-89-3, symbol Regulator_Linear:L78L05_SOT89
- removed U2, U3: TD7590_2, Package_TO_SOT_SMD:TO-263-5_TabPin3, symbol Regulator_Switching:TD7590_2
Connections:
- net labels removed: +5V, +5VL, +9V, 5V_HP, 5V_LP, 9V_HP, 9V_HP_EN, BAT1_1S, BAT1_2S, BAT1_3S, BAT2_1S, BAT2_2S, BAT2_3S, BCKP_3S, BCKP_EN, GND, VCC
- wire segments 197 -> 0
