File: hardware/PCB/TFG_PCB/TFG_PCB.kicad_pcb (KiCad board)
At the start: 2 copper layers, 101 parts, among them IC1 MCP3021A0T-E_OT, J1 Conn_01x02_Male, J10 Conn_01x02_Male, J11 Conn_01x02_Male, J13 Conn_01x04_Male, J15 Conn_01x04_Male, J16 Conn_01x02_Male, J17 Conn_01x02_Male, J18 Raspberry_Pi_2_3, J19 Conn_01x02_Male, J2 Conn_01x04_Male, J20 Conn_01x05_Male, J21 Conn_01x02_Male, J22 Conn_01x02_Male, J23 Conn_01x05_Male, J24 Conn_01x02_Male, J3 Conn_01x04_Male, J4 Conn_01x02_Male, J5 Conn_01x04_Male, J6 Conn_01x02_Male, J7 Conn_01x02_Male, J8 Conn_01x04_Male, J9 Conn_01x02_Male, Q1 IRF540N, Q10 2N2219, Q11 2N2219, Q12 FDD6685, Q13 FDD8896-F085, Q14 FDD8896-F085, Q15 FDD6685, Q16 2N2219, Q2 FDD6685, Q3 FDD6685, Q4 2N7002, Q5 2N2219, Q6 FDD6685, Q7 FDD8896-F085, Q8 FDD8896-F085, Q9 FDD6685, U1 L78L05_SOT89, U2 TD7590_2, U3 TD7590_2, U4 CD74HC4067M

Commit message: Object driver and wall detection
Routing:
- net Net-(R11-Pad1): track 42.4 -> 45.3 mm
Changed lines of the file:
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@@
   (general
     (thickness 1.6)
-    (drawings 9)
-    (tracks 1162)
+    (drawings 11)
+    (tracks 1163)
     (zones 0)
     (modules 101)
@@
     (visible_elements FFFFFF7F)
     (pcbplotparams
-      (layerselection 0x010fc_ffffffff)
+      (layerselection 0x030fc_ffffffff)
       (usegerberextensions false)
       (usegerberattributes false)
@@
       (drillshape 0)
       (scaleselection 1)
-      (outputdirectory ""))
+      (outputdirectory "D:/TFG/test_1_tank_controls/hardware/PCB/TFG_PCB/gerber/"))
   )
   (net 0 "")
@@
     )
   )
+  (dimension 147.32 (width 0.12) (layer F.SilkS)
+    (gr_text "147.320 mm" (at 136.525 99.06 270) (layer F.SilkS)
+      (effects (font (size 1 1) (thickness 0.15)))
+    )
+    (feature1 (pts (xy 127.635 172.72) (xy 135.841421 172.72)))
+    (feature2 (pts (xy 127.635 25.4) (xy 135.841421 25.4)))
+    (crossbar (pts (xy 135.255 25.4) (xy 135.255 172.72)))
+    (arrow1a (pts (xy 135.255 172.72) (xy 134.668579 171.593496)))
+    (arrow1b (pts (xy 135.255 172.72) (xy 135.841421 171.593496)))
+    (arrow2a (pts (xy 135.255 25.4) (xy 134.668579 26.526504)))
+    (arrow2b (pts (xy 135.255 25.4) (xy 135.841421 26.526504)))
+  )
+  (dimension 92.075 (width 0.12) (layer F.SilkS)
+    (gr_text "92.075 mm" (at 81.5975 16.51) (layer F.SilkS)
+      (effects (font (size 1 1) (thickness 0.15)))
+    )
+    (feature1 (pts (xy 127.635 25.4) (xy 127.635 17.193579)))
+    (feature2 (pts (xy 35.56 25.4) (xy 35.56 17.193579)))
+    (crossbar (pts (xy 35.56 17.78) (xy 127.635 17.78)))
+    (arrow1a (pts (xy 127.635 17.78) (xy 126.508496 18.366421)))
+    (arrow1b (pts (xy 127.635 17.78) (xy 126.508496 17.193579)))
+    (arrow2a (pts (xy 35.56 17.78) (xy 36.686504 18.366421)))
+    (arrow2b (pts (xy 35.56 17.78) (xy 36.686504 17.193579)))
+  )
   (gr_text "Jorge Huete TFG 2019-2020" (at 81.28 135.255) (layer B.Mask)
     (effects (font (size 1 1) (thickness 0.15)) (justify mirror))
@@
   (segment (start 67.056 51.816) (end 67.056 51.816) (width 0.3) (layer F.Cu) (net 25))
   (via (at 67.056 51.816) (size 0.8) (drill 0.4) (layers F.Cu B.Cu) (net 25))
-  (segment (start 68.072 72.644) (end 68.072 72.644) (width 0.3) (layer F.Cu) (net 25))
   (via (at 67.056 56.27299) (size 0.8) (drill 0.4) (layers F.Cu B.Cu) (net 25))
   (segment (start 67.056 51.816) (end 67.056 56.27299) (width 0.3) (layer B.Cu) (net 25))
@@
   (segment (start 70.338356 87.040548) (end 70.338356 86.474863) (width 0.95) (layer B.Cu) (net 72))
   (segment (start 65.742294 111.853117) (end 66.307979 111.853117) (width 0.95) (layer B.Cu) (net 72))
+  (segment (start 68.674655 83.725345) (end 68.58 83.82) (width 0.7) (layer F.Cu) (net 72))
+  (segment (start 71.467506 83.725345) (end 68.674655 83.725345) (width 0.7) (layer F.Cu) (net 72))
   (segment (start 59.445 50.8) (end 64.200608 50.8) (width 0.65) (layer F.Cu) (net 73))
   (segment (start 64.200608 50.8) (end 71.975038 58.57443) (width 0.65) (layer F.Cu) (net 73))
